File: EMBEDDED SYSTEM ASSIGNMENT/EMBEDDED SYSTEM ASSIGNMENT.kicad_pcb (KiCad board)
At the start: 2 copper layers, 91.4 x 78.7 mm, 32 parts, among them J1 Battery, J10 Load Cell, J11 ESC, J12 To ESC, J2 Kill_Switch, J3 Buck_Out, J4 Buck_In, J5 WCS1700 Module, J6 Encoder Sensor, J7 Micro SD Card Reader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

Commit message: Final touches
Parts:
- J1: value Battery -> BATTERY
- J11: value ESC -> TO ESC
- J12: value To ESC -> TO ESC
- J3: value Buck_Out -> FROM BUCK
- J4: value Buck_In -> TO BUCK
Routing:
- net +16V: track 1.32 -> 43.9 mm, vias 0 -> 13
- net GND: vias 0 -> 118
- net Battery_+16V: vias 0 -> 6

Commit message: errors resolved
Parts:
- J1: value BATTERY -> Battery
- J11: value TO ESC -> ESC
- J12: value TO ESC -> To ESC
Changed lines of the file:
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@@
 			(net 32 "unconnected-(U1-D4-Pad5)")
 			(pinfunction "D4")
-			(pintype "bidirectional")
+			(pintype "bidirectional+no_connect")
 			(solder_mask_margin 0.102)
 		)
@@
 			(net 6 "unconnected-(U1-RX2-Pad6)")
 			(pinfunction "RX2")
-			(pintype "input")
+			(pintype "input+no_connect")
 			(solder_mask_margin 0.102)
 		)
@@
 			(net 12 "unconnected-(U1-TX2-Pad7)")
 			(pinfunction "TX2")
-			(pintype "output")
+			(pintype "output+no_connect")
 			(solder_mask_margin 0.102)
 		)
@@
 			(net 16 "unconnected-(U1-RX0-Pad12)")
 			(pinfunction "RX0")
-			(pintype "input")
+			(pintype "input+no_connect")
 			(solder_mask_margin 0.102)
 		)
@@
 			(net 24 "unconnected-(U1-TX0-Pad13)")
 			(pinfunction "TX0")
-			(pintype "output")
+			(pintype "output+no_connect")
 			(solder_mask_margin 0.102)
 		)
@@
 			(net 8 "unconnected-(U1-D34-Pad19)")
 			(pinfunction "D34")
-			(pintype "bidirectional")
+			(pintype "bidirectional+no_connect")
 			(solder_mask_margin 0.102)
 		)
@@
 			(net 14 "unconnected-(U1-D35-Pad20)")
 			(pinfunction "D35")
-			(pintype "bidirectional")
+			(pintype "bidirectional+no_connect")
 			(solder_mask_margin 0.102)
 		)
@@
 			(net 17 "unconnected-(U1-D32-Pad21)")
 			(pinfunction "D32")
-			(pintype "bidirectional")
+			(pintype "bidirectional+no_connect")
 			(solder_mask_margin 0.102)
 		)
@@
 			(net 19 "unconnected-(U1-D33-Pad22)")
 			(pinfunction "D33")
-			(pintype "bidirectional")
+			(pintype "bidirectional+no_connect")
 			(solder_mask_margin 0.102)
 		)
@@
 			(net 10 "unconnected-(U1-D25-Pad23)")
 			(pinfunction "D25")
-			(pintype "bidirectional")
+			(pintype "bidirectional+no_connect")
 			(solder_mask_margin 0.102)
 		)
@@
 			)
 		)
-		(property "Value" "BATTERY"
+		(property "Value" "Battery"
 			(at 3.6 4 0)
 			(layer "F.SilkS" knockout)
@@
 			)
 		)
-		(property "Value" "TO ESC"
+		(property "Value" "To ESC"
 			(at 3.6 4 90)
 			(layer "F.SilkS" knockout)
@@
 			)
 		)
-		(property "Value" "TO ESC"
+		(property "Value" "ESC"
 			(at 2.5 4.6 90)
 			(layer "F.SilkS" knockout)
