File: EMBEDDED SYSTEM ASSIGNMENT/EMBEDDED SYSTEM ASSIGNMENT.kicad_sch (KiCad schematic)
At the start: 32 parts, among them J1 Battery, J10 Load Cell, J11 ESC, J12 To ESC, J2 Kill_Switch, J3 Buck_Out, J4 Buck_In, J5 WCS1700 Module, J6 Encoder Sensor, J7 Micro SD Card Reader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

Commit message: errors resolved
Parts:
- J3: value Buck_Out -> FROM BUCK
- J4: value Buck_In -> TO BUCK
Connections:
- no-connect marks 10 -> 20
Changed lines of the file:
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@@
+	)
+	(no_connect
+		(at 88.9 193.04)
 	)
 	(no_connect
@@
 	)
 	(no_connect
+		(at 88.9 162.56)
+	)
+	(no_connect
 		(at 58.42 160.02)
+	)
+	(no_connect
+		(at 88.9 180.34)
 	)
 	(no_connect
@@
 	)
 	(no_connect
+		(at 88.9 195.58)
+	)
+	(no_connect
+		(at 88.9 167.64)
+	)
+	(no_connect
+		(at 58.42 177.8)
+	)
+	(no_connect
 		(at 58.42 162.56)
 	)
@@
 	)
 	(no_connect
+		(at 88.9 160.02)
+	)
+	(no_connect
 		(at 58.42 154.94)
 	)
@@
 	(no_connect
 		(at 36.83 185.42)
+	)
+	(no_connect
+		(at 88.9 190.5)
+	)
+	(no_connect
+		(at 88.9 170.18)
+	)
+	(no_connect
+		(at 88.9 187.96)
 	)
 	(wire
@@
 			)
 		)
-		(property "Value" "Buck_Out"
+		(property "Value" "FROM BUCK"
 			(at 107.95 96.5201 0)
 			(effects
@@
 			)
 		)
-		(property "Value" "Buck_In"
+		(property "Value" "TO BUCK"
 			(at 88.9 95.2501 0)
 			(effects
